Commit message: updated files with error correction

File: stereo_description/urdf/camera.xacro (robot description, xacro)
@@ -10,5 +10,5 @@
   <link name="stereo_cam">
     <collision>
-      <origin xyz="0 0 0" rpy="0 0 0"/>
+      <origin xyz="0 0 0" rpy="0 0 1.26"/>
       <geometry>
     <box size="0.1 0.1 0.1"/>
